File: controller_pcb/controller_pcb.kicad_pcb (KiCad board)
At the start: 2 copper layers, 24 x 22.1 mm, 17 parts, among them J1 IO connector, SW1 PEC11L-4220F-S0015, U1 ATtiny1606-M

Commit message: Loadsa updates
Parts:
- added J12: LED_Pins, Project:Mounting_Hole_Pattern, F.Cu at (50.8, 50.8)
- added R21: 220, Resistor_SMD:R_0603_1608Metric, F.Cu at (41.7, 48.5)
- TP11: renamed from TP1; footprint TestPoint:TestPoint_Pad_D1.5mm -> TestPoint:TestPoint_Pad_D1.0mm
- moved R14 25.6 mm to (54.6, 47.5)
- moved R12 25.6 mm to (56.4, 47.5)
- moved C12 25.5 mm to (54.6, 50.8)
- moved C13 25.5 mm to (56.4, 50.8)
- moved J11 25.4 mm to (45.7, 59.7)
- moved SW11 25.4 mm to (50.8, 50.8)
- moved C11 25.4 mm to (47.2, 52.1)
- moved R11 25.4 mm to (47.2, 55.1)
- moved U11 25.4 mm to (50.3, 52.1)
- moved R15 25.3 mm to (54.6, 54.1)
- moved R13 25.3 mm to (56.4, 54.1)
- moved TP11 25.2 mm to (49.0, 48.5)
- moved R17 24.9 mm to (56.1, 44.5), turned to 0 degrees
- moved R18 24.8 mm to (52.1, 42.7), turned to 0 degrees
- moved R19 24.7 mm to (47.8, 42.7), turned to 0 degrees
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- renumbered C1 to C11, C2 to C12, C3 to C13, J1 to J11, R10 to R11, R1 to R12, R3 to R13, R2 to R14, R4 to R15, R5 to R16, R6 to R17, R7 to R18, R8 to R19, R9 to R20, SW1 to SW11, U1 to U11
Connections:
- J11 pad 1: VCC -> GND
- J11 pad 2: GND -> VCC
- J11 pad 3: SCL -> INT
- J11 pad 5: INT -> SCL
- SW11 pad S1: ENCS -> GND
- SW11 pad S2: GND -> ENCS
- U11 pad 1: unconnected-(U1-PA2-Pad1) -> LED6
- U11 pad 10: unconnected-(U1-PB4-Pad10) -> LED1
- U11 pad 16: unconnected-(U1-PC1-Pad16) -> LED2
- U11 pad 17: unconnected-(U1-PC2-Pad17) -> LED3
- U11 pad 18: unconnected-(U1-PC3-Pad18) -> LED4
- U11 pad 20: unconnected-(U1-PA1-Pad20) -> LED5
Routing:
- net VCC: track 15.1 -> 35.9 mm
- net LED1: track 0.00 -> 13.9 mm, vias 0 -> 2
- net LED3: track 0.00 -> 9.97 mm
- net LED4: track 0.00 -> 9.34 mm
- net LED6: track 0.00 -> 8.35 mm
- net LED2: track 0.00 -> 7.92 mm
- net LED5: track 0.00 -> 7.61 mm
- net INT: track 12.8 -> 7.73 mm
- net ENCS: track 4.10 -> 8.73 mm, vias 0 -> 1
- net ENCB: track 2.56 -> 6.62 mm, vias 0 -> 2
- net ENCA: track 9.11 -> 5.09 mm
- net Net-(J12-Pin_1): track 0.00 -> 2.62 mm
- net GND: track 6.65 -> 9.04 mm, vias 0 -> 1
- net Net-(J12-Pin_5): track 0.00 -> 2.37 mm
- net Net-(J12-Pin_6): track 0.00 -> 2.15 mm
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Other:
- board text removed: "INT SDA SCL GND VCC"

Commit message: Almost done
Parts:
- J11: footprint Connector_PinHeader_2.54mm:PinHeader_1x05_P2.54mm_Vertical -> Project:Project_PinHeader_1x05_P2.54mm_Vertical
- SW11: footprint Rotary_Encoder:RotaryEncoder_Bourns_Vertical_PEC12R-3x17F-Sxxxx -> Project:Project_RotaryEncoder_Bourns_Vertical_PEC12R-3x17F-Sxxxx
- U11: footprint Package_DFN_QFN:VQFN-20-1EP_3x3mm_P0.4mm_EP1.7x1.7mm -> Project:Project_ATTINY1616_VQFN-20-1EP_3x3mm_P0.4mm_EP1.7x1.7mm
Changed lines of the file:
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@@
     (pad "6" thru_hole circle (at -9.049965 -5.225 150) (size 2 2) (drill 1) (layers "*.Cu" "*.Mask")
       (net 12 "Net-(J12-Pin_6)") (pinfunction "Pin_6") (pintype "passive"))
+    (model "${KICAD6_3DMODEL_DIR}/Connector_Pin.3dshapes/Pin_D1.0mm_L10.0mm.wrl"
+      (offset (xyz 6.142356 8.454228 -3.5))
+      (scale (xyz 1 1 1))
+      (rotate (xyz 0 0 0))
+    )
+    (model "${KICAD6_3DMODEL_DIR}/Connector_Pin.3dshapes/Pin_D1.0mm_L10.0mm.wrl"
+      (offset (xyz 2.172677 10.221642 -3.5))
+      (scale (xyz 1 1 1))
+      (rotate (xyz 0 0 0))
+    )
+    (model "${KICAD6_3DMODEL_DIR}/Connector_Pin.3dshapes/Pin_D1.0mm_L10.0mm.wrl"
+      (offset (xyz -2.172677 10.221642 -3.5))
+      (scale (xyz 1 1 1))
+      (rotate (xyz 0 0 0))
+    )
+    (model "${KICAD6_3DMODEL_DIR}/Connector_Pin.3dshapes/Pin_D1.0mm_L10.0mm.wrl"
+      (offset (xyz -6.142356 8.454228 -3.5))
+      (scale (xyz 1 1 1))
+      (rotate (xyz 0 0 0))
+    )
+    (model "${KICAD6_3DMODEL_DIR}/Connector_Pin.3dshapes/Pin_D1.0mm_L10.0mm.wrl"
+      (offset (xyz -9.049965 5.225 -3.5))
+      (scale (xyz 1 1 1))
+      (rotate (xyz 0 0 0))
+    )
+    (model "${KICAD6_3DMODEL_DIR}/Connector_Pin.3dshapes/Pin_D1.0mm_L10.0mm.wrl"
+      (offset (xyz 9.049965 5.225 -3.5))
+      (scale (xyz 1 1 1))
+      (rotate (xyz 0 0 0))
+    )
+    (model "/home/matti/devel/encodering/build/led_pcb.step"
+      (offset (xyz 0 0 -6.1))
+      (scale (xyz 1 1 1))
+      (rotate (xyz 180 0 0))
+    )
   )
   (footprint "Resistor_SMD:R_0603_1608Metric" (layer "F.Cu")
@@
     )
   )
-  (footprint "Package_DFN_QFN:VQFN-20-1EP_3x3mm_P0.4mm_EP1.7x1.7mm" (layer "F.Cu")
+  (footprint "Project:Project_ATTINY1616_VQFN-20-1EP_3x3mm_P0.4mm_EP1.7x1.7mm" (layer "F.Cu")
     (at 50.292 52.07)
     (descr "VQFN, 20 Pin (http://ww1.microchip.com/downloads/en/DeviceDoc/20%20Lead%20VQFN%203x3x0_9mm_1_7EP%20U2B%20C04-21496a.pdf), generated with kicad-footprint-generator ipc_noLead_generator.py")
@@
       ))
     (pad "2" smd roundrect (at -1.45 -0.4) (size 0.8 0.2) (layers "F.Cu" "F.Paste" "F.Mask") (roundrect_rratio 0.25)
-      (net 22 "unconnected-(U11-PA3-Pad2)") (pinfunction "PA3") (pintype "bidirectional"))
+      (net 22 "unconnected-(U11-PA3-Pad2)") (pinfunction "PA3") (pintype "bidirectional+no_connect"))
     (pad "3" smd roundrect (at -1.45 0) (size 0.8 0.2) (layers "F.Cu" "F.Paste" "F.Mask") (roundrect_rratio 0.25)
       (net 7 "GND") (pinfunction "GND") (pintype "power_in"))
@@
       ))
     (pad "6" smd custom (at -0.8 1.45) (size 0.143431 0.143431) (layers "F.Cu" "F.Paste" "F.Mask")
-      (net 23 "unconnected-(U11-PA5-Pad6)") (pinfunction "PA5") (pintype "bidirectional") (thermal_bridge_angle 90)
+      (net 23 "unconnected-(U11-PA5-Pad6)") (pinfunction "PA5") (pintype "bidirectional+no_connect") (thermal_bridge_angle 90)
       (options (clearance outline) (anchor circle))
       (primitives
@@
       (net 10 "INT") (pinfunction "PA6") (pintype "bidirectional"))
     (pad "8" smd roundrect (at 0 1.45) (size 0.2 0.8) (layers "F.Cu" "F.Paste" "F.Mask") (roundrect_rratio 0.25)
-      (net 26 "unconnected-(U11-PA7-Pad8)") (pinfunction "PA7") (pintype "bidirectional"))
+      (net 26 "unconnected-(U11-PA7-Pad8)") (pinfunction "PA7") (pintype "bidirectional+no_connect"))
     (pad "9" smd roundrect (at 0.4 1.45) (size 0.2 0.8) (layers "F.Cu" "F.Paste" "F.Mask") (roundrect_rratio 0.25)
-      (net 27 "unconnected-(U11-PB5-Pad9)") (pinfunction "PB5") (pintype "bidirectional"))
+      (net 27 "unconnected-(U11-PB5-Pad9)") (pinfunction "PB5") (pintype "bidirectional+no_connect"))
     (pad "10" smd custom (at 0.8 1.45) (size 0.143431 0.143431) (layers "F.Cu" "F.Paste" "F.Mask")
       (net 19 "LED1") (pinfunction "PB4") (pintype "bidirectional") (thermal_bridge_angle 90)
@@
       ))
     (pad "12" smd roundrect (at 1.45 0.4) (size 0.8 0.2) (layers "F.Cu" "F.Paste" "F.Mask") (roundrect_rratio 0.25)
-      (net 28 "unconnected-(U11-PB2-Pad12)") (pinfunction "PB2") (pintype "bidirectional"))
+      (net 28 "unconnected-(U11-PB2-Pad12)") (pinfunction "PB2") (pintype "bidirectional+no_connect"))
     (pad "13" smd roundrect (at 1.45 0) (size 0.8 0.2) (layers "F.Cu" "F.Paste" "F.Mask") (roundrect_rratio 0.25)
       (net 9 "SDA") (pinfunction "PB1") (pintype "bidirectional"))
@@
     (pad "21" smd rect (at 0 0) (size 1.7 1.7) (layers "F.Cu" "F.Mask")
       (net 7 "GND") (pinfunction "GND") (pintype "passive"))
-    (model "${KICAD6_3DMODEL_DIR}/Package_DFN_QFN.3dshapes/VQFN-20-1EP_3x3mm_P0.4mm_EP1.7x1.7mm.wrl"
-      (offset (xyz 0 0 0))
-      (scale (xyz 1 1 1))
-      (rotate (xyz 0 0 0))
+    (model "${KICAD6_3DMODEL_DIR}/Package_DFN_QFN.3dshapes/VQFN-20-1EP_3x3mm_P0.4mm_EP1.7x1.7mm.wrl" hide
+      (offset (xyz 0 0 0))
+      (scale (xyz 1 1 1))
+      (rotate (xyz 0 0 0))
+    )
+    (model "ATTINY1616-MFR--3DModel-STEP-510211.STEP"
+      (offset (xyz 0 0 0))
+      (scale (xyz 1 1 1))
+      (rotate (xyz -90 0 0))
     )
   )
@@
     )
   )
-  (footprint "Connector_PinHeader_2.54mm:PinHeader_1x05_P2.54mm_Vertical" (layer "F.Cu")
+  (footprint "Project:Project_PinHeader_1x05_P2.54mm_Vertical" (layer "F.Cu")
     (at 45.72 59.69 90)
     (descr "Through hole straight pin header, 1x05, 2.54mm pitch, single row")
@@
     )
   )
-  (footprint "Rotary_Encoder:RotaryEncoder_Bourns_Vertical_PEC12R-3x17F-Sxxxx" (layer "B.Cu")
+  (footprint "Project:Project_RotaryEncoder_Bourns_Vertical_PEC12R-3x17F-Sxxxx" (layer "B.Cu")
     (at 50.8 50.8 180)
     (descr "Bourns rotary encoder, PEC12R, with switch, with bushing, vertical shaft, 17.5mm shaft, https://www.bourns.com/docs/product-datasheets/pec12r.pdf")
@@
     (pad "SH" thru_hole oval (at 0 -5.6 180) (size 4.1 3) (drill oval 3.1 2) (layers "*.Cu" "*.Mask"))
     (pad "SH" thru_hole oval (at 0 5.6 180) (size 4.1 3) (drill oval 3.1 2) (layers "*.Cu" "*.Mask"))
-    (model "${KICAD7_3DMODEL_DIR}/Rotary_Encoder.3dshapes/RotaryEncoder_Bourns_Vertical_PEC12R-3x17F-Sxxxx.wrl"
+    (model "${KICAD7_3DMODEL_DIR}/Rotary_Encoder.3dshapes/RotaryEncoder_Bourns_Vertical_PEC12R-3x17F-Sxxxx.wrl" hide
       (offset (xyz -7.5 2.5 0))
       (scale (xyz 1 1 1))
       (rotate (xyz 0 0 0))
     )
-  )
+    (model "PEC11L-4220F-S0015--3DModel-STEP-269445.STEP"
+      (offset (xyz 0 0 0))
+      (scale (xyz 1 1 1))
+      (rotate (xyz -90 0 90))
+    )
+  )
