File: controller_pcb/controller_pcb.kicad_sch (KiCad schematic)
At the start: 18 parts, among them J1 IO connector, J2 LED pins, SW1 PEC11L-4220F-S0015, U1 ATtiny1606-M

Commit message: LED ring generator 2.0 + kigen fixes
Parts:
- U1: LCSC (none) -> pollo
- renumbered C2 to C1
Changed lines of the file:
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@@
     (pin "1")
     (instances
-      (project "encodering"
+      (project "controller_pcb"
         (path "/512aed83-5f66-45ea-b2c1-65299dbb2e35"
           (reference "R6") (unit 1)
@@
     (pin "1")
     (instances
-      (project "encodering"
+      (project "controller_pcb"
         (path "/512aed83-5f66-45ea-b2c1-65299dbb2e35"
           (reference "#PWR02") (unit 1)
@@
     (pin "1")
     (instances
-      (project "encodering"
+      (project "controller_pcb"
         (path "/512aed83-5f66-45ea-b2c1-65299dbb2e35"
           (reference "#PWR07") (unit 1)
@@
     (pin "1")
     (instances
-      (project "encodering"
+      (project "controller_pcb"
         (path "/512aed83-5f66-45ea-b2c1-65299dbb2e35"
           (reference "R1") (unit 1)
@@
     (pin "1")
     (instances
-      (project "encodering"
+      (project "controller_pcb"
         (path "/512aed83-5f66-45ea-b2c1-65299dbb2e35"
           (reference "R2") (unit 1)
@@
     (pin "4")
     (instances
-      (project "encodering"
+      (project "controller_pcb"
         (path "/512aed83-5f66-45ea-b2c1-65299dbb2e35"
           (reference "J2") (unit 1)
@@
     (pin "1")
     (instances
-      (project "encodering"
+      (project "controller_pcb"
         (path "/512aed83-5f66-45ea-b2c1-65299dbb2e35"
           (reference "#PWR04") (unit 1)
@@
     (pin "1")
     (instances
-      (project "encodering"
+      (project "controller_pcb"
         (path "/512aed83-5f66-45ea-b2c1-65299dbb2e35"
           (reference "TP1") (unit 1)
@@
     (pin "1")
     (instances
-      (project "encodering"
+      (project "controller_pcb"
         (path "/512aed83-5f66-45ea-b2c1-65299dbb2e35"
           (reference "#PWR08") (unit 1)
@@
     (pin "1")
     (instances
-      (project "encodering"
+      (project "controller_pcb"
         (path "/512aed83-5f66-45ea-b2c1-65299dbb2e35"
           (reference "R9") (unit 1)
@@
     (pin "1")
     (instances
-      (project "encodering"
+      (project "controller_pcb"
         (path "/512aed83-5f66-45ea-b2c1-65299dbb2e35"
           (reference "R10") (unit 1)
@@
     (pin "1")
     (instances
-      (project "encodering"
+      (project "controller_pcb"
         (path "/512aed83-5f66-45ea-b2c1-65299dbb2e35"
           (reference "#PWR011") (unit 1)
@@
     (pin "1")
     (instances
-      (project "encodering"
+      (project "controller_pcb"
         (path "/512aed83-5f66-45ea-b2c1-65299dbb2e35"
           (reference "R7") (unit 1)
@@
     (pin "1")
     (instances
-      (project "encodering"
+      (project "controller_pcb"
         (path "/512aed83-5f66-45ea-b2c1-65299dbb2e35"
           (reference "#PWR012") (unit 1)
@@
     (pin "1")
     (instances
-      (project "encodering"
+      (project "controller_pcb"
         (path "/512aed83-5f66-45ea-b2c1-65299dbb2e35"
           (reference "R3") (unit 1)
@@
     (pin "S1")
     (instances
-      (project "encodering"
+      (project "controller_pcb"
         (path "/512aed83-5f66-45ea-b2c1-65299dbb2e35"
           (reference "SW1") (unit 1)
@@
   (symbol (lib_id "Device:C") (at 125.73 71.755 180) (unit 1)
     (in_bom yes) (on_board yes) (dnp no)
-    (property "Reference" "C2" (at 129.54 70.485 0)
+    (property "Reference" "C1" (at 129.54 70.485 0)
       (effects (font (size 1.27 1.27)) (justify right))
     )
@@
     (pin "1")
     (instances
-      (project "encodering"
-        (path "/512aed83-5f66-45ea-b2c1-65299dbb2e35"
-          (reference "C2") (unit 1)
+      (project "controller_pcb"
+        (path "/512aed83-5f66-45ea-b2c1-65299dbb2e35"
+          (reference "C1") (unit 1)
         )
       )
@@
     (pin "1")
     (instances
-      (project "encodering"
+      (project "controller_pcb"
         (path "/512aed83-5f66-45ea-b2c1-65299dbb2e35"
           (reference "R4") (unit 1)
@@
     (pin "1")
     (instances
-      (project "encodering"
+      (project "controller_pcb"
         (path "/512aed83-5f66-45ea-b2c1-65299dbb2e35"
           (reference "C3") (unit 1)
@@
     (pin "1")
     (instances
-      (project "encodering"
+      (project "controller_pcb"
         (path "/512aed83-5f66-45ea-b2c1-65299dbb2e35"
           (reference "#PWR03") (unit 1)
@@
     (pin "1")
     (instances
-      (project "encodering"
+      (project "controller_pcb"
         (path "/512aed83-5f66-45ea-b2c1-65299dbb2e35"
           (reference "#PWR09") (unit 1)
@@
     (pin "1")
     (instances
-      (project "encodering"
+      (project "controller_pcb"
         (path "/512aed83-5f66-45ea-b2c1-65299dbb2e35"
           (reference "#PWR010") (unit 1)
@@
     (pin "1")
     (instances
-      (project "encodering"
+      (project "controller_pcb"
         (path "/512aed83-5f66-45ea-b2c1-65299dbb2e35"
           (reference "#PWR05") (unit 1)
@@
     (pin "1")
     (instances
-      (project "encodering"
+      (project "controller_pcb"
         (path "/512aed83-5f66-45ea-b2c1-65299dbb2e35"
           (reference "R8") (unit 1)
@@
     (pin "1")
     (instances
-      (project "encodering"
+      (project "controller_pcb"
         (path "/512aed83-5f66-45ea-b2c1-65299dbb2e35"
           (reference "#PWR06") (unit 1)
@@
     (pin "2")
     (instances
-      (project "encodering"
+      (project "controller_pcb"
         (path "/512aed83-5f66-45ea-b2c1-65299dbb2e35"
           (reference "J1") (unit 1)
@@
     (pin "1")
     (instances
-      (project "encodering"
+      (project "controller_pcb"
         (path "/512aed83-5f66-45ea-b2c1-65299dbb2e35"
           (reference "#PWR01") (unit 1)
@@
     (pin "1")
     (instances
-      (project "encodering"
+      (project "controller_pcb"
         (path "/512aed83-5f66-45ea-b2c1-65299dbb2e35"
           (reference "C1") (unit 1)
@@
     (pin "1")
     (instances
-      (project "encodering"
+      (project "controller_pcb"
         (path "/512aed83-5f66-45ea-b2c1-65299dbb2e35"
           (reference "R5") (unit 1)
@@
     )
     (property "Datasheet" "http://ww1.microchip.com/downloads/en/DeviceDoc/ATtiny806_1606_Data_Sheet_40002029A.pdf" (at 48.26 81.28 0)
+      (effects (font (size 1.27 1.27)) hide)
+    )
+    (property "LCSC" "pollo" (at 48.26 81.28 0)
       (effects (font (size 1.27 1.27)) hide)
     )
@@
     (pin "10")
     (instances
-      (project "encodering"
+      (project "controller_pcb"
         (path "/512aed83-5f66-45ea-b2c1-65299dbb2e35"
           (reference "U1") (unit 1)
@@
     )
     (instances
-      (project "encodering"
+      (project "controller_pcb"
         (path "/512aed83-5f66-45ea-b2c1-65299dbb2e35" (page "2"))
       )

Commit message: Loadsa updates
Parts:
- removed J2: LED pins, Connector_PinHeader_1.27mm:PinHeader_1x05_P1.27mm_Vertical, symbol Connector_Generic:Conn_01x05
- added J12: LED_Pins, Project:Mounting_Hole_Pattern, symbol Connector_Generic:Conn_01x06
- added R21: 220, Resistor_SMD:R_0603_1608Metric, symbol Device:R
- TP11: renamed from TP1; footprint TestPoint:TestPoint_Pad_D1.5mm -> TestPoint:TestPoint_Pad_D1.0mm
- renumbered C1 to C11, C1 to C12, C3 to C13, J1 to J11, R10 to R11, R1 to R12, R3 to R13, R2 to R14, R4 to R15, R5 to R16, R6 to R17, R7 to R18, R8 to R19, R9 to R20, SW1 to SW11, U1 to U11
Connections:
- net ENCS: now also SW11.S2; no longer SW11.S1
- net GND: now also J11.1 (Pin_1), SW11.S1; no longer J11.2 (Pin_2), SW11.S2
- net INT: now also J11.3 (Pin_3); no longer J11.5 (Pin_5)
- net LED1: now also U11.10 (PB4)
- net LED2: now also U11.16 (PC1)
- net LED3: now also U11.17 (PC2)
- net LED4: now also U11.18 (PC3)
- net LED5: now also U11.20 (PA1)
- net SCL: now also J11.5 (Pin_5); no longer J11.3 (Pin_3)
- net VCC: now also J11.2 (Pin_2); no longer J11.1 (Pin_1)
- net at R17.2: now also J12.2 (Pin_2)
- net at R16.2: now also J12.1 (Pin_1)
- net at R18.2: now also J12.3 (Pin_3)
- net at R19.2: now also J12.4 (Pin_4)
- net at R20.2: now also J12.5 (Pin_5)
- net LED6: now reaches U11.1 (PA2)
- net LED6: now also R21.1
- new net: J12.6 (Pin_6), R21.2
- no-connect marks 5 -> 1
Other:
- removed sheet Untitled Sheet
- moved on the sheet: C12, C13, R12, R13, R14, R15, SW11

Commit message: Almost done
Parts:
- J11: footprint Connector_PinHeader_2.54mm:PinHeader_1x05_P2.54mm_Vertical -> Project:Project_PinHeader_1x05_P2.54mm_Vertical
- SW11: footprint Rotary_Encoder:RotaryEncoder_Bourns_Vertical_PEC12R-3x17F-Sxxxx -> Project:Project_RotaryEncoder_Bourns_Vertical_PEC12R-3x17F-Sxxxx
- U11: footprint Package_DFN_QFN:VQFN-20-1EP_3x3mm_P0.4mm_EP1.7x1.7mm -> Project:Project_ATTINY1616_VQFN-20-1EP_3x3mm_P0.4mm_EP1.7x1.7mm
Connections:
- no-connect marks 1 -> 5
Other:
- moved on the sheet: C12, C13, J11, J12, R11, R12, R13, R14, R15, R16, R17, R18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

Commit message: v1 for manufacturing
Parts:
- C2: renamed from C11; LCSC (none) -> C14663
- C3: renamed from C13; LCSC (none) -> C57112
- C4: renamed from C12; LCSC (none) -> C57112
- J2: renamed from J11; now left out of the parts list
- J3: renamed from J12; now left out of the parts list
- R10: renamed from R18; value 220 -> 20ohm; LCSC (none) -> C22950
- R11: renamed from R17; value 220 -> 20ohm; LCSC (none) -> C22950
- R12: renamed from R16; value 220 -> 20ohm; LCSC (none) -> C22950
- R2: renamed from R11; LCSC (none) -> C25804
- R3: renamed from R13; LCSC (none) -> C25804
- R4: renamed from R12; LCSC (none) -> C25804
- R5: renamed from R15; LCSC (none) -> C25804
- R6: renamed from R14; LCSC (none) -> C25804
- R7: renamed from R21; value 220 -> 20ohm; LCSC (none) -> C22950
- R8: renamed from R20; value 220 -> 20ohm; LCSC (none) -> C22950
- R9: renamed from R19; value 220 -> 20ohm; LCSC (none) -> C22950
- SW2: renamed from SW11; now left out of the parts list
- TP2: renamed from TP11; now left out of the parts list
- U2: renamed from U11; LCSC pollo -> C507118
Connections:
- net INT: now also J2.5 (Pin_5); no longer J2.3 (Pin_3)
- net LED1: now also R7.1, U2.2 (PA3); no longer R12.1, U2.10 (PB4)
- net LED2: now also R8.1, U2.1 (PA2); no longer R11.1, U2.16 (PC1)
- net LED3: now also R9.1, U2.20 (PA1); no longer R10.1, U2.17 (PC2)
- net LED4: now also R10.1; no longer R9.1
- net LED5: now also R11.1, U2.17 (PC2); no longer R8.1, U2.20 (PA1)
- net LED6: now also R12.1, U2.16 (PC1); no longer R7.1, U2.1 (PA2)
- net SCL: now also J2.4 (Pin_4); no longer J2.5 (Pin_5)
- net SDA: now also J2.3 (Pin_3); no longer J2.4 (Pin_4)
- net at J3.1 (Pin_1): now also R7.2; no longer R12.2
- net at J3.2 (Pin_2): now also R8.2; no longer R11.2
- net at J3.3 (Pin_3): now also R9.2; no longer R10.2
- net at J3.4 (Pin_4): now also R10.2; no longer R9.2
- net at J3.5 (Pin_5): now also R11.2; no longer R8.2
- net at J3.6 (Pin_6): now also R12.2; no longer R7.2
Other:
- moved on the sheet: R10, R11, R12, R7, R8, R9

Commit message: ACTUAL manufactured version
Parts:
- U1: renamed from U2; JLCPCB_CORRECTION (none) -> 0;0;270
- renumbered C2 to C1, C3 to C2, C4 to C3, J2 to J1, J3 to J2, R2 to R1, R11 to R10, R12 to R11, R3 to R2, R4 to R3, R5 to R4, R6 to R5, R7 to R6, R8 to R7, R9 to R8, R10 to R9, SW2 to SW1, TP2 to TP1

Commit message: Color
Other:
- moved on the sheet: C1, C2, C3, J1, J2, R1, R10, R11, R2, R3, R4, R5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
